File: switch.brd (EAGLE design)
At the start: 42.9 x 29.2 mm, 5 parts

Commit message: verze s hall snimacem
Connections:
- net N$4 renamed GPIO2
- net N$5 renamed GPIO0
Changed lines of the file:
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@@
 <?xml version="1.0" encoding="utf-8"?>
 <!DOCTYPE eagle SYSTEM "eagle.dtd">
-<eagle version="7.3.0">
+<eagle version="7.7.0">
 <drawing>
 <settings>
@@
 <wire x1="15.24" y1="7.62" x2="33.655" y2="7.62" width="0.4064" layer="16"/>
 </signal>
-<signal name="N$4">
+<signal name="GPIO2">
 <contactref element="SL1" pad="1"/>
 <contactref element="U$1" pad="P$7"/>
 <wire x1="15.24" y1="10.16" x2="7.62" y2="10.16" width="0.4064" layer="16"/>
 </signal>
-<signal name="N$5">
+<signal name="GPIO0">
 <contactref element="SL1" pad="3"/>
 <contactref element="U$1" pad="P$6"/>
