File: switch.sch (EAGLE design)
At the start: 5 parts

Commit message: verze s hall snimacem
Connections:
- net N$4 renamed GPIO2
- net N$5 renamed GPIO0
Changed lines of the file:
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@@
 <?xml version="1.0" encoding="utf-8"?>
 <!DOCTYPE eagle SYSTEM "eagle.dtd">
-<eagle version="7.3.0">
+<eagle version="7.7.0">
 <drawing>
 <settings>
@@
 </segment>
 </net>
-<net name="N$4" class="0">
+<net name="GPIO2" class="0">
 <segment>
 <pinref part="SL1" gate="-1" pin="S"/>
@@
 </segment>
 </net>
-<net name="N$5" class="0">
+<net name="GPIO0" class="0">
 <segment>
 <pinref part="SL1" gate="-3" pin="S"/>
